File: pcb/unflying-fish-controller/unflying-fish-controller.kicad_pcb (KiCad board)
At the start: 2 copper layers, 115 x 100 mm, 33 parts, among them J1 GY-NEO6MV2 (GPS), J10 SERVO, J11 SERVO, J12 NEOPIXEL, J13 DM3D-SF, J14 LM2596S (buck converter), J15 XL4016 (Buck Converter for Se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, J2 SS49E (Hall Effect Sensor), J3 MMC5603 (IMU), J4 GY-MS5837 (MAGENTOMETER), J5 ESC CAN, J8 SERVO, J9 SERVO, U1 ESP32-S3-DEVKITC-1-N16R8V, U2 LSM6DSOTR, U3 74AHCT125S14-13

Commit message: compact pcb slightly
Parts:
- moved J11 26.0 mm to (198.0, 135.0)
- moved J8 13.5 mm to (120.0, 137.0)
- moved J9 9.67 mm to (139.5, 136.5)
- moved J10 8.54 mm to (164.5, 137.0)
- moved J1 5.51 mm to (176.0, 75.5)
Routing:
- net /+6V: track 94.3 -> 131.0 mm
- net /SERVO4: track 78.3 -> 96.0 mm
- net /SERVO3: track 77.4 -> 71.5 mm
- net /GPS_TXD: track 208.3 -> 202.9 mm
- net /SERVO2: track 38.5 -> 33.5 mm
- net /SERVO1: track 40.7 -> 45.0 mm
- net /+5V: track 262.6 -> 258.9 mm
- net /GPS_RXD: track 164.3 -> 162.4 mm
- net GND: vias 154 -> 153
Other:
- board size 115 x 100 mm -> 114.9 x 89.5 mm

Commit message: add motor+driver for ballast
Parts:
- added C11: 0.1uF, Capacitor_THT:C_Disc_D5.0mm_W2.5mm_P2.50mm, F.Cu at (177.0, 62.0)
- added C12: 10nF, Capacitor_THT:C_Disc_D5.0mm_W2.5mm_P2.50mm, F.Cu at (169.0, 66.2)
- added C13: 2.2uF, Capacitor_THT:C_Disc_D5.0mm_W2.5mm_P2.50mm, F.Cu at (183.5, 68.2)
- added C14: 10uF, Capacitor_THT:CP_Radial_D5.0mm_P2.00mm, F.Cu at (180.0, 76.0)
- added J6: motor2, Connector_PinHeader_2.54mm:PinHeader_1x02_P2.54mm_Vertical, F.Cu at (166.3, 75.5)
- added J7: motor1, Connector_PinHeader_2.54mm:PinHeader_1x02_P2.54mm_Vertical, F.Cu at (171.7, 75.5)
- added R8: 10k, Resistor_THT:R_Axial_DIN0207_L6.3mm_D2.5mm_P7.62mm_Horizontal, F.Cu at (157.7, 71.0)
- added U4: DRV8833PW, afishthatdoesntfly:PW16_TEX, F.Cu at (176.5, 67.0)
- moved J1 28.5 mm to (204.5, 76.5)
Connections:
- U1 pad J1_16: unconnected-(U1-GPIO10-PadJ1_16) -> /BIN1
- U1 pad J1_7: unconnected-(U1-GPIO7-PadJ1_7) -> /AIN2
- U1 pad J3_18: unconnected-(U1-GPIO21-PadJ3_18) -> /AIN1
- U1 pad J3_4: unconnected-(U1-GPIO1-PadJ3_4) -> /BIN2
Routing:
- net /+6V: track 131.0 -> 373.8 mm
- net 3V3: track 185.8 -> 345.0 mm, vias 1 -> 3
- net /BIN1: track 0.00 -> 149.8 mm, vias 0 -> 2
- net /AIN2: track 0.00 -> 147.3 mm, vias 0 -> 1
- net /SERVO4: track 96.0 -> 206.6 mm, vias 0 -> 2
- net /HALL_OUT: track 122.9 -> 224.1 mm, vias 0 -> 1
- net /GPS_TXD: track 202.9 -> 106.8 mm
- net /AIN1: track 0.00 -> 94.5 mm, vias 0 -> 3
- net /NEO_IN: track 84.9 -> 167.4 mm
- net /SDA: track 111.4 -> 189.9 mm
- net /BIN2: track 0.00 -> 77.5 mm
- net /+5V: track 258.9 -> 330.4 mm
- net /ESC_SIG: track 55.0 -> 119.0 mm
- net /SCL: track 113.6 -> 177.5 mm, vias 2 -> 3
- net /SD_CS: track 65.2 -> 128.3 mm
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