File: pcb/unflying-fish-controller/unflying-fish-controller.kicad_sch (KiCad schematic)
At the start: 0 parts

Commit message: pcb!!!
Parts:
- added BT2: Battery, TerminalBlock:TerminalBlock_MaiXu_MX126-5.0-02P_1x02_P5.00mm, symbol Device:Battery
- added C1: 100uF, Capacitor_THT:CP_Radial_D6.3mm_P2.50mm, symbol Device:C
- added C10, C4: 1000uF, Capacitor_THT:CP_Radial_D10.0mm_P5.00mm, symbol Device:C
- added C2, C7, C9: 100nF, Capacitor_THT:C_Disc_D5.0mm_W2.5mm_P2.50mm, symbol Device:C
- added C3: 470uF C, Capacitor_THT:CP_Radial_D8.0mm_P3.50mm, symbol Device:C
- added C5, C6: 100nf, Capacitor_THT:C_Disc_D5.0mm_W2.5mm_P2.50mm, symbol Device:C
- added C8: 4.7uF, Capacitor_THT:CP_Radial_D5.0mm_P2.00mm, symbol Device:C
- added J1: GY-NEO6MV2 (GPS), Unflying Fish:GY-GPS6MV2, symbol Connector:Conn_01x04_Pin
- added J10, J11, J8, J9: SERVO, Connector_PinHeader_2.54mm:PinHeader_1x03_P2.54mm_Vertical, symbol Connector:Conn_01x03_Pin
- added J12: NEOPIXEL, Connector_PinHeader_2.54mm:PinHeader_1x03_P2.54mm_Vertical, symbol Connector:Conn_01x03_Pin
- added J13: DM3D-SF, Unflying Fish:CONN8_DM3D-SF_HIR, symbol DM3D-SF:DM3D-SF
- added J14: LM2596S (buck converter), Connector_PinHeader_2.54mm:PinHeader_1x04_P2.54mm_Vertical, symbol Connector:Conn_01x04_Pin
- added J15: XL4016 (Buck Converter for Servos), Connector_PinHeader_2.54mm:PinHeader_1x04_P2.54mm_Vertical, symbol Connector:Conn_01x04_Pin
- added J2: SS49E (Hall Effect Sensor), Connector_PinHeader_2.54mm:PinHeader_1x03_P2.54mm_Vertical, symbol Connector:Conn_01x03_Pin
- added J3: MMC5603 (IMU), Connector_PinHeader_2.54mm:PinHeader_1x05_P2.54mm_Vertical, symbol Connector:Conn_01x05_Pin
- added J4: GY-MS5837 (MAGENTOMETER), Connector_PinHeader_2.54mm:PinHeader_1x04_P2.54mm_Vertical, symbol Connector:Conn_01x04_Pin
- added J5: ESC CAN, Connector_PinHeader_2.54mm:PinHeader_1x02_P2.54mm_Vertical, symbol Connector:Conn_01x02_Pin
- added R1, R2: 4.7K, Resistor_THT:R_Axial_DIN0207_L6.3mm_D2.5mm_P7.62mm_Horizontal, symbol Device:R
- added R3, R4, R5: 10k, Resistor_THT:R_Axial_DIN0207_L6.3mm_D2.5mm_P7.62mm_Horizontal, symbol Device:R
- added R6: 330, Resistor_THT:R_Axial_DIN0207_L6.3mm_D2.5mm_P7.62mm_Horizontal, symbol Device:R
- added U1: ESP32-S3-DEVKITC-1-N16R8V, Unflying Fish:ESP32-S3-DEVKITC-1-N16R8V, symbol ESP32-S3-DEVKITC-1-N16R8V:ESP32-S3-DEVKITC-1-N16R8V
- added U2: LSM6DSOTR, Unflying Fish:LSM6DSOTR, symbol LSM6DSOTR:LSM6DSOTR
- added U3: 74AHCT125S14-13, Unflying Fish:74AHCT125S14-13, symbol 74AHCT125S14-13:74AHCT125S14-13
Connections:
- new net +5V: C10.1, C2.1, C3.1, C9.1, J1.1 (Pin_1), J12.1 (Pin_1), J14.3 (Pin_3), U1.J1_21 (5V0), U3.10 (*3OE), U3.13 (*4OE), U3.14 (VCC), U3.4 (*2OE)
- new net +6V: C4.1, J10.1 (Pin_1), J11.1 (Pin_1), J15.3 (Pin_3), J8.1 (Pin_1), J9.1 (Pin_1)
- new net 3V3: C1.1, C5.2, C6.2, C7.1, C8.1, J13.4, J2.1 (Pin_1), J3.1 (Pin_1), J4.1 (Pin_1), R1.1, R2.1, R3.2, R4.2, R5.2, U1.J1_1 (3V3), U1.J1_2 (3V3), U2.12 (CS), U2.5 (VDDIO), U2.8 (VDD)
- new net BATT+: BT2.1 (+), J14.1 (Pin_1), J15.1 (Pin_1)
- new net ESC_SIG: J5.1 (Pin_1), U1.J1_5 (GPIO5)
- new net GND: BT2.2 (-), C1.2, C10.2, C2.2, C3.2, C4.2, C5.1, C6.1, C7.2, C8.2, C9.2, J1.4 (Pin_4), J10.3 (Pin_3), J11.3 (Pin_3), J12.3 (Pin_3), J13.6, J14.2 (Pin_2), J14.4 (Pin_4), J15.2 (Pin_2), J15.4 (Pin_4), J2.2 (Pin_2), J3.3 (Pin_3), J4.2 (Pin_2), J5.2 (Pin_2), J8.3 (Pin_3), J9.3 (Pin_3), U1.J1_22 (GND), U1.J3_1 (GND), U1.J3_21 (GND), U1.J3_22 (GND), U2.1 (SDO/SA0), U2.2 (SDx), U2.3 (SCx), U2.6 (GND), U2.7 (GND), U3.1 (*1OE), U3.12 (4A), U3.5 (2A), U3.7 (GND), U3.9 (3A)
- new net GPS_RXD: J1.2 (Pin_2), U1.J1_10 (GPIO17)
- new net GPS_TXD: J1.3 (Pin_3), U1.J1_11 (GPIO18)
- new net HALL_OUT: J2.3 (Pin_3), U1.J1_4 (GPIO4)
- new net NEO_DIN: J12.2 (Pin_2), R6.2
- new net NEO_IN: U1.J1_6 (GPIO6), U3.2 (1A)
- new net NEO_OUT: R6.1, U3.3 (1Y)
- new net SCL: J3.4 (Pin_4), J4.3 (Pin_3), R2.2, U1.J1_15 (GPIO9), U2.13 (SCL)
- new net SDA: J3.5 (Pin_5), J4.4 (Pin_4), R1.2, U1.J1_12 (GPIO8), U2.14 (SDA)
- new net SD_CS: J13.2, R3.1, U1.J1_20 (GPIO14)
- new net SD_DAT1: J13.8, R4.1
- new net SD_DAT2: J13.1, R5.1
- new net SD_MISO: J13.7, U1.J1_19 (GPIO13)
- new net SD_MOSI: J13.3, U1.J1_17 (GPIO11)
- new net SD_SCK: J13.5, U1.J1_18 (GPIO12)
- new net SERVO1: J8.2 (Pin_2), U1.J3_17 (GPIO47)
- new net SERVO2: J9.2 (Pin_2), U1.J3_16 (GPIO48)
- new net SERVO3: J10.2 (Pin_2), U1.J1_8 (GPIO15)
- new net SERVO4: J11.2 (Pin_2), U1.J1_9 (GPIO16)
- no-connect marks 0 -> 30
Other:
- note added: "ESP32"
- note added: "EVERYTHING ELSE"
- note added: "IMU"
- note added: "LED"
- note added: "MicroSD"
- note added: "POWER"

Commit message: add motor+driver for ballast
Parts:
- added C11: 0.1uF, Capacitor_THT:C_Disc_D5.0mm_W2.5mm_P2.50mm, symbol Device:C
- added C12: 10nF, Capacitor_THT:C_Disc_D5.0mm_W2.5mm_P2.50mm, symbol Device:C
- added C13: 2.2uF, Capacitor_THT:C_Disc_D5.0mm_W2.5mm_P2.50mm, symbol Device:C
- added C14: 10uF, Capacitor_THT:CP_Radial_D5.0mm_P2.00mm, symbol Device:C
- added J6: motor2, Connector_PinHeader_2.54mm:PinHeader_1x02_P2.54mm_Vertical, symbol Connector:Conn_01x02_Pin
- added J7: motor1, Connector_PinHeader_2.54mm:PinHeader_1x02_P2.54mm_Vertical, symbol Connector:Conn_01x02_Pin
- added R8: 10k, Resistor_THT:R_Axial_DIN0207_L6.3mm_D2.5mm_P7.62mm_Horizontal, symbol Device:R
- added U4: DRV8833PW, afishthatdoesntfly:PW16_TEX, symbol DRV8833PW:DRV8833PW
Connections:
- net +6V: now also C11.2, C12.1, C14.1, U4.12 (VM)
- net 3V3: now also R8.1, U4.1 (NSLEEP)
- net GND: now also C11.1, C13.1, C14.2, U4.13 (GND), U4.3 (AISEN), U4.6 (BISEN)
- net BIN1: now reaches U1.J1_16 (GPIO10)
- net BIN1: now also U4.9 (BIN1)
- net AIN2: now reaches U1.J1_7 (GPIO7)
- net AIN2: now also U4.15 (AIN2)
- net AIN1: now reaches U1.J3_18 (GPIO21)
- net AIN1: now also U4.16 (AIN1)
- net BIN2: now reaches U1.J3_4 (GPIO1)
- net BIN2: now also U4.10 (BIN2)
- new net AOUT1: J7.1 (Pin_1), U4.2 (AOUT1)
- new net AOUT2: J7.2 (Pin_2), U4.4 (AOUT2)
- new net BOUT1: J6.1 (Pin_1), U4.7 (BOUT1)
- new net BOUT2: J6.2 (Pin_2), U4.5 (BOUT2)
- new net NFAULT: R8.2, U4.8 (NFAULT)
- new net VCP: C12.2, U4.11 (VCP)
- new net VINT: C13.2, U4.14 (VINT)
- no-connect marks 30 -> 26
Other:
- moved on the sheet: J10, J11, J8, J9
